Commit message: standardize naming of new fanuc arm

File: jrl/urdfs/fanuc_R2000iC-165F_rtu/fanuc_R2000iC-165F_rtu.urdf (robot description, URDF)
Before this commit: robot R-2000iC 165F w RTU, 12 links, 11 joints
Links:
- link fanuc_base: geometry collision mesh filename=urdfs/fanuc_R2000iC-165F_rtu/geometry/collision/base.dae; visual mesh filename=urdfs/fanuc_R2000iC-165F_rtu/geometry/visual/base.dae
- link link_1: geometry collision mesh filename=urdfs/fanuc_R2000iC-165F_rtu/geometry/collision/link_1.dae; visual mesh filename=urdfs/fanuc_R2000iC-165F_rtu/geometry/visual/link_1.dae
- link link_2: geometry collision mesh filename=urdfs/fanuc_R2000iC-165F_rtu/geometry/collision/link_2.dae; visual mesh filename=urdfs/fanuc_R2000iC-165F_rtu/geometry/visual/link_2.dae
- link link_3: geometry collision mesh filename=urdfs/fanuc_R2000iC-165F_rtu/geometry/collision/link_3.dae; visual mesh filename=urdfs/fanuc_R2000iC-165F_rtu/geometry/visual/link_3.dae
- link link_4: geometry collision mesh filename=urdfs/fanuc_R2000iC-165F_rtu/geometry/collision/link_4.dae; visual mesh filename=urdfs/fanuc_R2000iC-165F_rtu/geometry/visual/link_4.dae
- link link_5: geometry collision mesh filename=urdfs/fanuc_R2000iC-165F_rtu/geometry/collision/link_5.dae; visual mesh filename=urdfs/fanuc_R2000iC-165F_rtu/geometry/visual/link_5.dae
- link link_6: geometry collision mesh filename=urdfs/fanuc_R2000iC-165F_rtu/geometry/collision/link_6.dae; visual mesh filename=urdfs/fanuc_R2000iC-165F_rtu/geometry/visual/link_6.dae
- link slide: geometry collision mesh filename=urdfs/fanuc_R2000iC-165F_rtu/geometry/collision/rtu_slide.s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; visual mesh filename=urdfs/fanuc_R2000iC-165F_rtu/geometry/visual/rtu_slide.stl
- link slide_base: geometry collision mesh filename=urdfs/fanuc_R2000iC-165F_rtu/geometry/collision/slide_base.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; visual mesh filename=urdfs/fanuc_R2000iC-165F_rtu/geometry/visual/slide_base.stl
